Commit message: Flip joint5 on irb140

File: drake/examples/IRB140/urdf/irb_140.urdf (robot description, URDF)
Before this commit: robot IRB140_-_M2004C_Complete_base.SLDASM, 7 links, 6 joints
Joints:
- joint joint5: axis 0 0 -1 -> 0 0 1

Commit message: Update joint limit to be slightly more conservative on joint 5

File: drake/examples/IRB140/urdf/irb_140.urdf (robot description, URDF)
Before this commit: robot IRB140_-_M2004C_Complete_base.SLDASM, 7 links, 6 joints
Joints:
- joint joint5: limit lower=-2.09439510 upper=2.09439510 effort=300 velocity=5.58 -> lower=-1.74 upper=1.74 effort=300 velocity=5.58
