Commit message: Added some hand-fit ground truth, some real data, and code for fitting a filter.

File: drake/examples/GelsightPerception/urdf/legobrickend.urdf (robot description, URDF)
Before this commit: robot justabox, 1 links, 0 joints
Links:
- link base_link: geometry collision box size=.80 .96 2.0; visual box size=.80 .96 2.0
